File: electronics/beacon/beacon.kicad_pcb (KiCad board)
At the start: 2 copper layers, 24 x 9.6 mm, 15 parts, among them J1 CONN_01X04, J2 CONN_01X04, J3 Rails, Q1 Q_NMOS_GSD, U1 ATTINY45-20XUR, U2 TPS70928DBV

Commit message: electronics: beacon: Improve schematic labeling & readability
Parts:
- D2: value Rectifier -> BAS4002A
- J1: value CONN_01X04 -> ICSP
- J2: value CONN_01X04 -> GPIO
- J3: value Rails -> RAILS
- Q1: value Q_NMOS_GSD -> 2N7002E
Connections:
- net Net-(C1-Pad1) renamed VCC
- net Net-(D2-Pad2) renamed /RAIL_R
- net Net-(D2-Pad3) renamed /RAIL_L
Changed lines of the file:
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@@
   (net 12 /PB3)
   (net 13 /PB4)
-  (net 14 "Net-(C1-Pad1)")
-  (net 15 "Net-(D2-Pad2)")
-  (net 16 "Net-(D2-Pad3)")
+  (net 14 VCC)
+  (net 15 /RAIL_L)
+  (net 16 /RAIL_R)
   (net_class Default "This is the default net class."
     (clearance 0.2)
@@
     (add_net /PB3)
     (add_net /PB4)
+    (add_net /RAIL_L)
+    (add_net /RAIL_R)
     (add_net /SCK)
     (add_net /~RST)
@@
     (add_net "Net-(U2-Pad3)")
     (add_net "Net-(U2-Pad4)")
+    (add_net VCC)
   )
   (net_class Power ""
@@
     (uvia_drill 0.1)
     (add_net GND)
-    (add_net "Net-(C1-Pad1)")
     (add_net "Net-(D1-Pad1)")
     (add_net "Net-(D1-Pad2)")
-    (add_net "Net-(D2-Pad2)")
-    (add_net "Net-(D2-Pad3)")
   )
   (net_class Tight ""
@@
       (effects (font (size 0.6 0.6) (thickness 0.1)))
     )
-    (fp_text value Rectifier (at -0.28 2.48 180) (layer F.Fab)
+    (fp_text value BAS4002A (at -0.28 2.48 180) (layer F.Fab)
       (effects (font (size 1 1) (thickness 0.15)))
     )
@@
       (net 1 GND))
     (pad 2 smd rect (at -1.1 0.95 90) (size 1 1.4) (layers F.Cu F.Paste F.Mask)
-      (net 15 "Net-(D2-Pad2)"))
+      (net 16 /RAIL_R))
     (pad 3 smd rect (at 1.1 0.95 90) (size 1 1.4) (layers F.Cu F.Paste F.Mask)
-      (net 16 "Net-(D2-Pad3)"))
+      (net 15 /RAIL_L))
     (pad 4 smd rect (at 1.1 -0.95 90) (size 1 1.4) (layers F.Cu F.Paste F.Mask)
-      (net 14 "Net-(C1-Pad1)"))
+      (net 14 VCC))
     (model TO_SOT_Packages_SMD.3dshapes/SOT-143.wrl
       (at (xyz 0 -0 0))
@@
       (effects (font (size 0.6 0.6) (thickness 0.1)))
     )
-    (fp_text value Q_NMOS_GSD (at 0 2.5) (layer F.Fab)
+    (fp_text value 2N7002E (at 0 2.5) (layer F.Fab)
       (effects (font (size 1 1) (thickness 0.15)))
     )
@@
     (fp_line (start 0.9 -1.55) (end 0.9 1.55) (layer F.Fab) (width 0.1))
     (pad 1 smd rect (at -1.1 -0.95) (size 1.06 0.65) (layers F.Cu F.Paste F.Mask)
-      (net 14 "Net-(C1-Pad1)"))
+      (net 14 VCC))
     (pad 2 smd rect (at -1.1 0) (size 1.06 0.65) (layers F.Cu F.Paste F.Mask)
       (net 1 GND))
@@
     (fp_line (start 1.4 0.65) (end -1.4 0.65) (layer F.CrtYd) (width 0.05))
     (pad 1 smd rect (at -0.75 0 270) (size 0.8 0.75) (layers F.Cu F.Paste F.Mask)
-      (net 14 "Net-(C1-Pad1)"))
+      (net 14 VCC))
     (pad 2 smd rect (at 0.75 0 270) (size 0.8 0.75) (layers F.Cu F.Paste F.Mask)
       (net 1 GND))
@@
       (effects (font (size 1 1) (thickness 0.15)) (justify mirror))
     )
-    (fp_text value CONN_01X04 (at -1 -5.5 90) (layer B.Fab)
+    (fp_text value ICSP (at -1 -5.5 90) (layer B.Fab)
       (effects (font (size 1 1) (thickness 0.15)) (justify mirror))
     )
@@
       (effects (font (size 1 1) (thickness 0.15)) (justify mirror))
     )
-    (fp_text value CONN_01X04 (at -1 -5.5 270) (layer B.Fab)
+    (fp_text value GPIO (at -1 -5.5 270) (layer B.Fab)
       (effects (font (size 1 1) (thickness 0.15)) (justify mirror))
     )
@@
       (effects (font (size 1 1) (thickness 0.15)))
     )
-    (fp_text value Rails (at 0 2.54) (layer F.Fab)
+    (fp_text value RAILS (at 0 2.54) (layer F.Fab)
       (effects (font (size 1 1) (thickness 0.15)))
     )
     (pad 1 smd rect (at -10 0) (size 4 2.4) (layers F.Cu F.Mask)
-      (net 16 "Net-(D2-Pad3)"))
+      (net 15 /RAIL_L))
     (pad 2 smd rect (at 10 0) (size 4 2.4) (layers F.Cu F.Mask)
-      (net 15 "Net-(D2-Pad2)"))
+      (net 16 /RAIL_R))
     (pad "" np_thru_hole circle (at 0 0) (size 1 1) (drill 1) (layers *.Cu *.Mask))
   )
@@
   (segment (start 145.75 108.95) (end 144.8 108) (width 0.4) (layer F.Cu) (net 14))
   (segment (start 151.5 107.05) (end 150.2 107.05) (width 0.4) (layer F.Cu) (net 14))
-  (segment (start 160 105) (end 158.870836 105) (width 0.4) (layer F.Cu) (net 15))
-  (segment (start 158.870836 105) (end 157.447223 103.576387) (width 0.4) (layer F.Cu) (net 15))
-  (segment (start 154.2 103.6) (end 153.4 104.4) (width 0.4) (layer F.Cu) (net 15))
-  (segment (start 153.4 104.4) (end 150.732002 104.4) (width 0.4) (layer F.Cu) (net 15))
-  (segment (start 150.732002 104.4) (end 150.332002 104) (width 0.4) (layer F.Cu) (net 15))
-  (segment (start 150.332002 104) (end 149.667998 104) (width 0.4) (layer F.Cu) (net 15))
-  (segment (start 148.3 107.05) (end 148.3 105.367998) (width 0.4) (layer F.Cu) (net 15))
-  (segment (start 148.3 105.367998) (end 149.667998 104) (width 0.4) (layer F.Cu) (net 15))
-  (segment (start 157.4 103.529164) (end 157.447223 103.576387) (width 0.4) (layer F.Cu) (net 15))
-  (segment (start 157.4 103.5) (end 157.4 103.529164) (width 0.4) (layer F.Cu) (net 15))
-  (segment (start 154.2 103.6) (end 157.42361 103.6) (width 0.4) (layer B.Cu) (net 15))
-  (segment (start 157.42361 103.6) (end 157.447223 103.576387) (width 0.4) (layer B.Cu) (net 15))
-  (via (at 157.447223 103.576387) (size 0.6) (drill 0.4) (layers F.Cu B.Cu) (net 15))
-  (via (at 154.2 103.6) (size 0.6) (drill 0.4) (layers F.Cu B.Cu) (net 15))
-  (segment (start 140 105) (end 144.95 105) (width 0.4) (layer F.Cu) (net 16))
-  (segment (start 144.95 105) (end 146.1 106.15) (width 0.4) (layer F.Cu) (net 16))
-  (segment (start 146.1 106.15) (end 146.1 107.05) (width 0.4) (layer F.Cu) (net 16))
+  (segment (start 140 105) (end 144.95 105) (width 0.4) (layer F.Cu) (net 15))
+  (segment (start 144.95 105) (end 146.1 106.15) (width 0.4) (layer F.Cu) (net 15))
+  (segment (start 146.1 106.15) (end 146.1 107.05) (width 0.4) (layer F.Cu) (net 15))
+  (segment (start 160 105) (end 158.870836 105) (width 0.4) (layer F.Cu) (net 16))
+  (segment (start 158.870836 105) (end 157.447223 103.576387) (width 0.4) (layer F.Cu) (net 16))
+  (segment (start 154.2 103.6) (end 153.4 104.4) (width 0.4) (layer F.Cu) (net 16))
+  (segment (start 153.4 104.4) (end 150.732002 104.4) (width 0.4) (layer F.Cu) (net 16))
+  (segment (start 150.732002 104.4) (end 150.332002 104) (width 0.4) (layer F.Cu) (net 16))
+  (segment (start 150.332002 104) (end 149.667998 104) (width 0.4) (layer F.Cu) (net 16))
+  (segment (start 148.3 107.05) (end 148.3 105.367998) (width 0.4) (layer F.Cu) (net 16))
+  (segment (start 148.3 105.367998) (end 149.667998 104) (width 0.4) (layer F.Cu) (net 16))
+  (segment (start 157.4 103.529164) (end 157.447223 103.576387) (width 0.4) (layer F.Cu) (net 16))
+  (segment (start 157.4 103.5) (end 157.4 103.529164) (width 0.4) (layer F.Cu) (net 16))
+  (segment (start 154.2 103.6) (end 157.42361 103.6) (width 0.4) (layer B.Cu) (net 16))
+  (segment (start 157.42361 103.6) (end 157.447223 103.576387) (width 0.4) (layer B.Cu) (net 16))
+  (via (at 157.447223 103.576387) (size 0.6) (drill 0.4) (layers F.Cu B.Cu) (net 16))
+  (via (at 154.2 103.6) (size 0.6) (drill 0.4) (layers F.Cu B.Cu) (net 16))
   (zone (net 1) (net_name GND) (layer F.Cu) (hatch edge 0.508)
     (connect_pads (clearance 0.25))
