File: electronics/locomotive_tof_sensor/locomotive_tof_sensor.kicad_pcb (KiCad board)
At the start: 2 copper layers, 10 x 8 mm, 6 parts, among them J1 TOF, U1 VL6180X

Commit message: electronics: locomotive_tof_sensor: Board Rev 1.0
Parts:
- added J2: INT, Measurement_Points:Measurement_Point_Square-SMD-Pad_Small, F.Cu at (145.8, 98.0)
- moved J1 0.25 mm to (150.0, 100.2), turned to 0 degrees
Routing:
- net +2V8: track 0.00 -> 20.6 mm, vias 0 -> 1
- net GND: track 0.00 -> 11.6 mm, vias 0 -> 1
- net /SCL: track 0.00 -> 7.30 mm, vias 0 -> 1
- net /INT: track 0.00 -> 3.26 mm
- net Net-(R1-Pad2): track 0.00 -> 1.91 mm
- net /SDA: track 0.00 -> 1.50 mm, vias 0 -> 1
- added copper zone on B.Cu, net GND
- added copper zone on F.Cu, net GND
Other:
- board size 10 x 8 mm -> 10 x 6 mm
- board text added: "INT"
- board text added: "JST-GH"
- board text added: "Rev 1.0"
- board text added: "bcan TOF"
