File: electronics/locomotive/connectors.sch (KiCad schematic (older format))
At the start: 7 parts, among them J1 JTAG, J2 USB_OTG, J3 CONN_01X32, J4 CONN_01X32, J5 TRAIN, J6 IR, J7 TOF

Commit message: electronics: locomotive: Board Rev 1.0
Parts:
- removed J3, J4: CONN_01X32, symbol CONN_01X32
- removed J5: TRAIN, symbol CONN_01X08
- added J3: PIN[1..16], Pin_Headers:Pin_Header_Straight_1x16_Pitch2.00mm, symbol CONN_01X16
- added J4: PIN[17..32], Pin_Headers:Pin_Header_Straight_1x16_Pitch2.00mm, symbol CONN_01X16
- added J5: PIN[49..64], Pin_Headers:Pin_Header_Straight_1x16_Pitch2.00mm, symbol CONN_01X16
- added J6: PIN[33..48], Pin_Headers:Pin_Header_Straight_1x16_Pitch2.00mm, symbol CONN_01X16
- added J7: TRAIN, Pin_Headers:Pin_Header_Straight_2x04_Pitch2.54mm_SMD, symbol CONN_02X04
- J1: footprint (none) -> Pin_Headers:Pin_Header_Straight_2x05_Pitch1.27mm_SMD
- J2: footprint (none) -> Connectors_Molex:USB_Micro-B_Molex_47346-0001
- J8: renamed from J6; footprint (none) -> Connectors_JST:JST_GH_SM04B-GHS-TB_04x1.25mm_Angled
- J9: renamed from J7; footprint (none) -> Connectors_JST:JST_GH_SM04B-GHS-TB_04x1.25mm_Angled
Connections:
- net labels added: BOOT0, F-, Io, M+, M-, NRST, R-, T+, T-, USB_VBUS, VBAT
- net labels removed: +5V, 5V, PA[0..15], PB[0..15], PC[0..15]
- wire segments 70 -> 104
Other:
- note removed: "F-"
- note removed: "I_0"
- note removed: "M+"
- note removed: "M-"
- note removed: "R-"
- note removed: "T+"
- note removed: "T-"
- moved on the sheet: J1, J2, J8, J9
