File: electronics/locomotive/locomotive.sch (KiCad schematic (older format))
At the start: 8 parts, among them U2 M95512-RDW6TP, U6 6N136

Commit message: electronics: locomotive: Board Rev 1.0
Parts:
- removed D3: 1N4148, symbol D
- removed R19: 1k5, symbol R
- removed R20: 10k, symbol R
- removed R21: 10k (not fitted), symbol R
- removed U6: 6N136, DIP-8, symbol 6N136
- added C13: 2u2, Capacitors_SMD:C_0603, symbol C_Small
- added D1: CDBHM240L-HF, bcan:TO-269AA, symbol D_Bridge_+-AA
- added D2: CUS08F30, Diodes_SMD:D_SOD-323, symbol D_Small
- added D3: 1N4148, Diodes_SMD:D_SOD-523, symbol D_Small
- added J1: PIN[1..32], bcan:Castellations_1x32_Pitch2.00mm, symbol CONN_01X32
- added J2: PIN[33..64], bcan:Castellations_1x32_Pitch2.00mm, symbol CONN_01X32
- added J3: JTAG, Pin_Headers:Pin_Header_Straight_2x05_Pitch1.27mm_SMD, symbol CONN_02X05
- added J4: USB_OTG, bcan:USB_Micro-B_Amphenol_10118192, symbol USB_OTG
- added J5: RAILS, bcan:Castellations_1x02_Pitch2.00mm, symbol CONN_01X02
- added J6: MOTOR, bcan:Castellations_1x02_Pitch2.00mm, symbol CONN_01X02
- added J7: TRAIN, Pin_Headers:Pin_Header_Straight_2x04_Pitch2.54mm_SMD, symbol CONN_02X04
- added J8: IR, Connectors_JST:JST_GH_BM04B-GHS-TBT_04x1.25mm_Straight, symbol CONN_01X04
- added J9: TOF, Connectors_JST:JST_GH_SM04B-GHS-TB_04x1.25mm_Angled, symbol CONN_01X04
- added JP5: USB_VBUS, bcan:Solder_Jumper_NC, symbol Jumper_NC_Small
- added Q1, Q2: MMBT2222A, TO_SOT_Packages_SMD:SOT-23, symbol Q_NPN_BEC
- added Q3, Q4: DMG6601LVT, TO_SOT_Packages_SMD:SOT-23-6, symbol Q_DUAL_NMOS_PMOS_G1S2G2D2S1D1
- added R12, R20: 10k, Resistors_SMD:R_0603, symbol R_Small
- added R13: 33k2, Resistors_SMD:R_0603, symbol R_Small
- added R14: 26k1, Resistors_SMD:R_0603, symbol R_Small
- added R15, R16: 1k, Resistors_SMD:R_0603, symbol R_Small
- added R17, R18: 100, Resistors_SMD:R_2512, symbol R_Small
- added R19: 1k5, Resistors_SMD:R_0603, symbol R_Small
- added R4: 13k3, Resistors_SMD:R_0603, symbol R_Small
- added R5: 2k8, Resistors_SMD:R_0603, symbol R_Small
- added R8, R9: 4k7, Resistors_SMD:R_0603, symbol R_Small
- added U5: SPX3819M5, TO_SOT_Packages_SMD:SOT-23-5, symbol SPX3819M5
- added U7: TLP293, Housings_SSOP:SOP-4_4.4x2.8mm_Pitch1.27mm, symbol TLP291
- R10, R11: footprint (none) -> Resistors_SMD:R_0603
- U2: footprint (none) -> Housings_SSOP:TSSOP-8_4.4x3mm_Pitch0.65mm
Connections:
- net +2V8: now also C13.1, J1.12 (P12), J1.13 (P13), J2.15 (P15), J2.16 (P16), J3.1 (P1), J8.1 (P1), J9.1 (P1), R13.1, R20.1, R8.1, R9.1, U5.5 (OUT)
- net +5V: now also D2.2 (A), J1.32 (P32), J4.1 (VBUS), JP5.1, R12.1
- net GND: now also C13.2, D1.2 (-), J1.18 (P18), J1.19 (P19), J2.31 (P31), J2.32 (P32), J3.3 (P3), J3.5 (P5), J3.7 (P7), J3.9 (P9), J4.5 (GND), J4.6 (shield), J8.4 (P4), J9.4 (P4), Q1.2 (E), Q2.2 (E), Q3.5 (S), Q4.5 (S), R12.2, R14.2, R5.2, U5.2 (GND), U7.3
- net MOT+: now also J6.1 (P1), J7.2 (P2), Q3.4 (D), Q3.6 (D)
- net MOT-: now also J5.2 (P2), J7.7 (P7), Q4.4 (D), Q4.6 (D)
- net RAIL_L: now also D1.4, D3.2 (A), J5.1 (P1), J7.8 (P8), U7.2
- net RAIL_R: now also D1.3, J6.2 (P2), J7.1 (P1), R19.2
- net VCC: now also D1.1 (+), D2.1 (K), J1.31 (P31), Q3.2 (S), Q4.2 (S), R17.1, R18.1, R4.1, U5.1 (IN), U5.3 (EN)
- net MISO renamed PB14
- net PB14: now also J2.3 (P3)
- net MOSI renamed PB15
- net PB15: now also J2.4 (P4)
- net NSS renamed PB12
- net PB12: now also J2.1 (P1)
- net SCK renamed PB13
- net PB13: now also J2.2 (P2)
- new net: D3.1 (K), R19.1, U7.1
- new net: R13.2, R14.1, U5.4 (ADJ)
- new net: Q2.1 (B), R16.1
- new net: Q1.1 (B), R15.1
- new net: Q2.3 (C), Q4.1 (G), Q4.3 (G), R18.2
- new net: Q1.3 (C), Q3.1 (G), Q3.3 (G), R17.2
- new net BOOT0: J2.28 (P28)
- new net FRONT-: J1.5 (P5), J7.5 (P5)
- new net NRST: J1.7 (P7), J3.10 (P10)
- new net PA0: J1.14 (P14)
- new net PA1: J1.15 (P15)
- new net PA10: J2.11 (P11), J4.2 (D-)
- new net PA11: J2.12 (P12), J4.3 (D+)
- new net PA12: J2.13 (P13), J4.4 (ID)
- new net PA13: J2.14 (P14), J3.2 (P2)
- new net PA14: J2.17 (P17), J3.4 (P4)
- new net PA15: J2.18 (P18), J3.8 (P8)
- new net PA2: J1.16 (P16)
- new net PA3: J1.17 (P17)
- new net PA4: J1.20 (P20)
- new net PA5: J1.21 (P21)
- new net PA6: J1.22 (P22)
- new net PA7: J1.23 (P23)
- new net PA8: J2.9 (P9)
- new net PA9: J2.10 (P10), JP5.2
- new net PB0: J1.26 (P26), J8.2 (P2)
- new net PB1: J1.27 (P27), J8.3 (P3)
- new net PB10: J1.29 (P29), J9.3 (P3), R8.2
- new net PB11: J1.30 (P30), J9.2 (P2), R9.2
- new net PB2: J1.28 (P28)
- new net PB3: J2.23 (P23), J3.6 (P6)
- new net PB4: J2.24 (P24)
- new net PB5: J2.25 (P25)
- new net PB6: J2.26 (P26)
- new net PB7: J2.27 (P27)
- new net PB8: J2.29 (P29), R15.2
- new net PB9: J2.30 (P30), R16.2
- new net PC0: J1.8 (P8)
- new net PC1: J1.9 (P9)
- new net PC10: J2.19 (P19)
- new net PC11: J2.20 (P20)
- new net PC12: J2.21 (P21)
- new net PC13: J1.2 (P2), R20.2, U7.4
- new net PC14: J1.3 (P3)
- new net PC15: J1.4 (P4)
- new net PC2: J1.10 (P10), R4.2, R5.1
- new net PC3: J1.11 (P11)
- new net PC4: J1.24 (P24)
- new net PC5: J1.25 (P25)
- new net PC6: J2.5 (P5)
- new net PC7: J2.6 (P6)
- new net PC8: J2.7 (P7)
- new net PC9: J2.8 (P8)
- new net PD2: J2.22 (P22)
- new net REAR-: J1.6 (P6), J7.4 (P4)
- new net TRAIN_I: J7.3 (P3)
- new net VBAT: J1.1 (P1)
Other:
- moved on the sheet: R10, R11, U2
